Commit message: 修复gui控制joint旋转时姿态跳变问题,原因为joint_state_publisher和joint_state_publisher_gui功能冲突,两者都发布joint_state消息;增加base_footprint link(可以认为是机器人底盘对地面的投影),解决当以base_link为基点时底盘一半陷入地底问题

File: zxz_ros_tools_ws/src/cpp07_urdf/urdf/urdf/demo04_basefootprint.urdf (robot description, URDF)
Before this commit: robot Lbot, 2 links, 1 joints
Links:
- added link base_footprint; visual sphere radius=0.01
Joints:
- added joint baselink2basefootprint: type fixed, parent base_footprint, child base_link, origin xyz=0.0 0.0 0.1 rpy=0.0 0.0 0.0
- joint camera2baselink: axis 0 0 1 -> 0.0 0.0 1.0
