Commit message: 添加仿真launch文件(通过文件包含启动gazebo,通过gazebo_ros entity在gazebo中加载机器人模型),修复robot_core中无轮胎bug(inertial标签必须在link标签内,否则gazebo中就无法加载该link)

File: articubot_ws/src/articubot/description/robot_core_back.xacro (robot description, xacro)
@@ -1,15 +1,18 @@
 <robot xmlns:xacro="http://www.ros.org/wiki/xacro">
     <xacro:include filename="inertial_macros.xacro"/>
-    <xacro:property name="chassis_length" value="0.3" />
-    <xacro:property name="chassis_width" value="0.3" />
-    <xacro:property name="chassis_height" value="0.15" />
-    <xacro:property name="chassis_mass" value="0.5" />
-    <xacro:property name="wheel_offset_y" value="0.175" />
-    <xacro:property name="wheel_radius" value="0.05" />
-    <xacro:property name="wheel_thickness" value="0.04" />
-    <xacro:property name="wheel_mass" value="0.1" />
-    <xacro:property name="caster_radius" value="0.05" />
-    <xacro:property name="caster_offset_x" value="0.24" />
-    <xacro:property name="caster_mass" value="0.1" />
+    <xacro:property name="chassis_length" value="0.335" />
+    <xacro:property name="chassis_width" value="0.265" />
+    <xacro:property name="chassis_height" value="0.138" />
+    <xacro:property name="chassis_mass" value="1.0" />
+    <xacro:property name="wheel_offset_x" value="0.226" />
+    <xacro:property name="wheel_offset_y" value="0.1485" />
+    <xacro:property name="wheel_offset_z" value="0.01" />
+    <xacro:property name="wheel_radius" value="0.033" />
+    <xacro:property name="wheel_thickness" value="0.026" />
+    <xacro:property name="wheel_mass" value="0.05" />
+    <xacro:property name="caster_radius" value="0.01" />
+    <xacro:property name="caster_offset_x" value="0.075" />
+    <xacro:property name="caster_offset_z" value="${wheel_offset_z - wheel_radius + caster_radius}" />
+    <xacro:property name="caster_mass" value="0.01" />
     <material name="white">
         <color rgba="1.0 1.0 1.0 1.0"/>
@@ -32,5 +35,5 @@
         <parent link="base_link"/>
         <child link="chassis"/>
-        <origin xyz="-0.1 0.0 0.0"/>
+        <origin xyz="${-wheel_offset_x} 0.0 ${-wheel_offset_z}"/>
     </joint>
     <!-- CHASSIS LINK -->
@@ -41,5 +44,5 @@
             </geometry>
             <origin xyz="${chassis_length/2} 0.0 ${chassis_height/2}"/>
-            <material name="white" />
+            <material name="orange" />
         </visual>
         <collision>
@@ -74,8 +77,8 @@
                 </geometry>
             </collision>
-            <xacro:inertial_cylinder mass="${wheel_mass}" radius="${wheel_radius}" length="${wheel_thickness}">
-                <origin xyz="0.0 0.0 0.0" rpy="0.0 0.0 0.0"/>
-            </xacro:inertial_cylinder>
         </link>
+        <xacro:inertial_cylinder mass="${wheel_mass}" radius="${wheel_radius}" length="${wheel_thickness}">
+            <origin xyz="0.0 0.0 0.0" rpy="0.0 0.0 0.0"/>
+        </xacro:inertial_cylinder>
     </xacro:macro>
     <!-- WHEEL LINK -->
@@ -86,5 +89,5 @@
         <parent link="chassis"/>
         <child link="caster_wheel"/>
-        <origin xyz="${caster_offset_x} 0.0 0.0"/>
+        <origin xyz="${caster_offset_x} 0.0 ${caster_offset_z}"/>
     </joint>
     <link name="caster_wheel">
