Commit message: 通过libgazebo_ros_diff_drive库实现两轮差速模型仿真

File: articubot_ws/src/articubot/description/robot.urdf.xacro (robot description, xacro)
@@ -1,3 +1,4 @@
 <robot xmlns:xacro="http://www.ros.org/wiki/xacro" name="robot">
     <xacro:include filename="robot_core.xacro"/>
+    <xacro:include filename="gazebo_control.xacro"/>
 </robot>

File: articubot_ws/src/articubot/description/robot_core.xacro (robot description, xacro)
@@ -41,5 +41,5 @@
             </geometry>
             <origin xyz="${chassis_length/2} 0.0 ${chassis_height/2}"/>
-            <material name="white" />
+            <material name="orange" />
         </visual>
         <collision>
@@ -53,4 +53,7 @@
         </xacro:inertial_box>
     </link>
+    <gazebo reference="chassis">
+        <material>Gazebo/Orange</material>
+    </gazebo>
     <!-- WHEEL FUNC -->
     <xacro:macro name="wheel_func" params="link_name left_flag">
@@ -82,4 +85,10 @@
     <xacro:wheel_func link_name="left_wheel" left_flag="1" />
     <xacro:wheel_func link_name="right_wheel" left_flag="-1" />
+    <gazebo reference="left_wheel">
+        <material>Gazebo/Blue</material>
+    </gazebo>
+    <gazebo reference="right_wheel">
+        <material>Gazebo/Blue</material>
+    </gazebo>
     <!-- CASTER LINK -->
     <joint name="caster_wheel_joint" type="fixed">
@@ -104,3 +113,8 @@
         </xacro:inertial_sphere>
     </link>
+    <gazebo reference="caster_wheel">
+        <material>Gazebo/Black</material>
+        <mu1 value="0.001"/>
+        <mu2 value="0.001"/>
+    </gazebo>
 </robot>
